File: usb cable tester.kicad_pcb (KiCad board)
At the start: 2 copper layers, 80.6 x 58.4 mm, 97 parts, among them J1 USB_C_all_pins, J2 USB3_B_Micro, J3 USB3_B, J4 USB3_A, J5 USB_C_all_pins, J6 USB_B_Mini

Commit message: Updated net names to make stuff more understanable
Connections:
- net Net-(J2-Pad4) renamed /OTG
- net Net-(J4-Pad1) renamed /VBUS_A4
- net Net-(J4-Pad2) renamed /D-_A7
- net Net-(J4-Pad3) renamed /D+_A6
- net Net-(J4-Pad4) renamed /GND_A1
- net Net-(J4-Pad5) renamed /RX1-_B10
- net Net-(J4-Pad6) renamed /RX1+_B11
- net Net-(J4-Pad7) renamed /DRAIN
- net Net-(J4-Pad8) renamed /TX1-_A3
- net Net-(J4-Pad9) renamed /TX1+_A2
- net Net-(J5-PadA10) renamed /RX2-_A10
- net Net-(J5-PadA11) renamed /RX2+_A11
- net Net-(J5-PadA12) renamed /GND_A12
- net Net-(J5-PadA8) renamed /SBU1_A8
- net Net-(J5-PadA9) renamed /VBUS_A9
- net Net-(J5-PadB1) renamed /GND_B1
- net Net-(J5-PadB12) renamed /GND_B12
- net Net-(J5-PadB2) renamed /TX2+_B2
- net Net-(J5-PadB3) renamed /TX2-_B3
- net Net-(J5-PadB4) renamed /VBUS_B4
- net Net-(J5-PadB5) renamed /CC2_B5
- net Net-(J5-PadB6) renamed /D+_B6
- net Net-(J5-PadB7) renamed /D-_B7
- net Net-(J5-PadB8) renamed /SBU2_B8
- net Net-(J5-PadB9) renamed /VBUS_B9
- J4 pad 10: Net-(J4-Pad10) -> /SHIELD_S1
- R26 pad 1: Net-(J4-Pad10) -> /SHIELD_S1
- R6 pad 1: Net-(J5-PadA5) -> /CC1_A5
Routing:
- net Net-(J4-Pad10): track 51.5 -> 0.06 mm, vias 8 -> 4
- net /SHIELD_S1: track 0.00 -> 51.5 mm, vias 0 -> 4
- net Net-(J5-PadA5): track 22.6 -> 0.00 mm
- net /CC1_A5: track 0.00 -> 22.6 mm
- added copper zone on B.Cu, net /SHIELD_S1
- added copper zone on F.Cu, net /SHIELD_S1
- removed copper zone on B.Cu, net Net-(J4-Pad10)
- removed copper zone on F.Cu, net Net-(J4-Pad10)

Commit message: Synced footprints and changed references
Parts:
- renumbered REF** to SYM1, REF** to SYM2, REF** to SYM3, REF** to SYM4, REF** to TOOLING1, REF** to TOOLING2, REF** to TOOLING3
Connections:
- J4 pad 10: /SHIELD_S1 -> /SHIELD
- J5 pad A5: Net-(J5-PadA5) -> /CC1_A5
- J5 pad S1: Net-(J4-Pad10) -> /SHIELD
- R26 pad 1: /SHIELD_S1 -> /SHIELD
Routing:
- net /SHIELD: track 0.00 -> 51.5 mm, vias 0 -> 8
- net /SHIELD_S1: track 51.5 -> 0.00 mm, vias 4 -> 0
- net Net-(J4-Pad10): track 0.06 -> 0.00 mm, vias 4 -> 0
- added copper zone on B.Cu, net /SHIELD
- added copper zone on F.Cu, net /SHIELD
- removed copper zone on B.Cu, net /SHIELD_S1
- removed copper zone on F.Cu, net /SHIELD_S1

Commit message: Change values of resistors and LEDs
Parts:
- D1: value DRAIN -> Red
- D10, D11: value D+ -> Red
- D12: value RX1- -> Red
- D13: value RX1+ -> Red
- D14: value TX1- -> Red
- D15: value TX1+ -> Red
- D16: value RX2- -> Red
- D17: value RX2+ -> Red
- D18: value TX2- -> Red
- D19: value TX2+ -> Red
- D2, D3, D4, D5: value VBUS -> Red
- D20: value SBU1 -> Red
- D21: value SBU2 -> Red
- D27: value OTG -> Red
- D6: value CC1 -> Red
- D7: value CC2 -> Red
- D8, D9: value D- -> Red
- R1, R10, R11, R12, R13, R14, R15, R16, R17, R18, R19, R2, R20, R21, R27, R3, R4, R5, R6, R7, R8, R9: value 470R -> 1k

Commit message: Fix values missed before, hide some stuff from BOM
Parts:
- D22, D23, D24, D25: value GND -> Red
- D26: value SHIELD -> Red
- R22, R23, R24, R25, R26: value 470R -> 1k
- SYM3: value cat -> (none)
Other:
- rule pad_to_mask_clearance: 0.05 -> 0
